Commit message: Added lidar tf.

File: go2_description/xacro/robot.xacro (robot description, xacro)
@@ -55,4 +55,11 @@
                 izz="${trunk_izz}"/>
         </inertial>
+    </link>
+    <joint name="lidar_joint" type="fixed">
+        <parent link="trunk"/>
+        <child link="utlidar_lidar"/>
+        <origin rpy="0 0 0" xyz="0.32715 -0.00003 -0.04297"/>
+    </joint>
+    <link name="utlidar_lidar">
     </link>
     <joint name="imu_joint" type="fixed">

Commit message: Accurate Lidar tf.

File: go2_description/xacro/robot.xacro (robot description, xacro)
@@ -59,5 +59,5 @@
         <parent link="trunk"/>
         <child link="utlidar_lidar"/>
-        <origin rpy="0 0 0" xyz="0.32715 -0.00003 -0.04297"/>
+        <origin rpy="0 -0.2 0" xyz="0.29515 -0.00003 -0.06597"/>
     </joint>
     <link name="utlidar_lidar">
